File: Hardware/Gamma_spectrometer.kicad_sch (KiCad schematic)
At the start: 47 parts, among them J1 Conn_01x04, J10 Test Pad, J11 Test Pad, J2 Conn_01x04, J3 Conn_01x01, J4 Conn_01x04, J5 Test Pad, J6 Test Pad, J7 Test Pad, J8 Test Pad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

Commit message: code stuff i guess
Parts:
- gave numbers to parts that had none: 1
Changed lines of the file:
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@@
   (symbol (lib_id "Connector:Conn_01x01_Female") (at 87.63 151.13 90) (unit 1)
     (in_bom yes) (on_board yes) (fields_autoplaced)
-    (property "Reference" "J?" (id 0) (at 88.9 150.4949 90)
+    (property "Reference" "J12" (id 0) (at 88.9 150.4949 90)
       (effects (font (size 1.27 1.27)) (justify right))
     )
@@
     )
     (path "/95cd8917-dd22-409d-9bf7-9fcc99b0bc9b"
-      (reference "J?") (unit 1) (value "Test Pad") (footprint "TestPoint:TestPoint_THTPad_1.0x1.0mm_Drill0.5mm")
+      (reference "J12") (unit 1) (value "Test Pad") (footprint "TestPoint:TestPoint_THTPad_1.0x1.0mm_Drill0.5mm")
     )
     (path "/e5f3c54b-7060-4a13-b929-4280c6a62fa5"

Commit message: fixed som BOM stuff
Parts:
- removed J1: Conn_01x04, Connector_PinHeader_2.00mm:PinHeader_1x04_P2.00mm_Vertical, symbol Connector_Generic:Conn_01x04
Other:
- note added: "Interupt"
- note added: "Micro Controller"
- note added: "Voltage Regulator"
- note removed: "Shift Register R-2R DAC"
- moved on the sheet: C1, C2, C3, C4, C5, D1, D2, J10, J11, J12, J2, J3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
